File: hardware/particulate-matter.kicad_pcb (KiCad board)
At the start: 2 copper layers, 70 x 40 mm, 35 parts, among them P1 CON-SENSOR2, P2 BOOT, P3 DEBUG, U1 XMC1404, U2 DRILL, U3 DRILL, U4 DRILL, U5 DRILL, U6 PMS7003, X1 16MHz

Commit message: Fix footprint
Parts:
- RP2: footprint 4X0402 -> kicad-libraries:4X0402
Changed lines of the file:
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@@
   (layers
     (0 F.Cu signal)
-    (31 B.Cu signal)
+    (31 B.Cu signal hide)
     (32 B.Adhes user)
     (33 F.Adhes user)
@@
       (xy 2.48217 3.513666) (xy 2.482863 3.409859) (xy 2.482863 3.409859)) (layer B.SilkS) (width 0.1))
   )
-  (module 4X0402 (layer F.Cu)
-    (at 156.3 78.4 90)
-    (attr smd)
-    (fp_text reference RP2 (at -0.025 0.25 90) (layer F.Fab)
-      (effects (font (size 0.2 0.2) (thickness 0.05)))
-    )
-    (fp_text value 100 (at -0.025 -0.45 90) (layer F.Fab)
-      (effects (font (size 0.2 0.2) (thickness 0.05)))
-    )
-    (fp_line (start -1.04902 -0.89916) (end 1.04902 -0.89916) (layer F.Fab) (width 0.001))
-    (fp_line (start 1.04902 -0.89916) (end 1.04902 0.89916) (layer F.Fab) (width 0.001))
-    (fp_line (start -1.04902 0.89916) (end 1.04902 0.89916) (layer F.Fab) (width 0.001))
-    (fp_line (start -1.04902 -0.89916) (end -1.04902 0.89916) (layer F.Fab) (width 0.001))
-    (pad 1 smd rect (at -0.7493 0.575 270) (size 0.29972 0.65) (layers F.Cu F.Paste F.Mask)
-      (net 52 "Net-(RP2-Pad1)"))
-    (pad 2 smd rect (at -0.24892 0.575 270) (size 0.29972 0.65) (layers F.Cu F.Paste F.Mask)
-      (net 30 PMS_RX))
-    (pad 3 smd rect (at 0.24892 0.575 270) (size 0.29972 0.65) (layers F.Cu F.Paste F.Mask)
-      (net 29 PMS_TX))
-    (pad 4 smd rect (at 0.7493 0.575 270) (size 0.29972 0.65) (layers F.Cu F.Paste F.Mask)
-      (net 53 "Net-(RP2-Pad4)"))
-    (pad 5 smd rect (at 0.7493 -0.575 90) (size 0.29972 0.65) (layers F.Cu F.Paste F.Mask)
-      (net 54 "Net-(RP2-Pad5)"))
-    (pad 6 smd rect (at 0.24892 -0.575 90) (size 0.29972 0.65) (layers F.Cu F.Paste F.Mask)
-      (net 57 "Net-(RP2-Pad6)"))
-    (pad 7 smd rect (at -0.24892 -0.575 90) (size 0.29972 0.65) (layers F.Cu F.Paste F.Mask)
-      (net 58 "Net-(RP2-Pad7)"))
-    (pad 8 smd rect (at -0.7493 -0.575 90) (size 0.29972 0.65) (layers F.Cu F.Paste F.Mask)
-      (net 55 "Net-(RP2-Pad8)"))
-    (model Resistors_SMD/R_4x0402.wrl
-      (at (xyz 0 0 0))
-      (scale (xyz 1 1 1))
-      (rotate (xyz 0 0 90))
-    )
-  )
   (module kicad-libraries:C0805 (layer F.Cu)
     (at 157.35 85.11 270)
@@
     )
   )
+  (module kicad-libraries:4X0402 (layer F.Cu)
+    (at 156.3 78.4 90)
+    (attr smd)
+    (fp_text reference RP2 (at -0.025 0.25 90) (layer F.Fab)
+      (effects (font (size 0.2 0.2) (thickness 0.05)))
+    )
+    (fp_text value 100 (at -0.025 -0.45 90) (layer F.Fab)
+      (effects (font (size 0.2 0.2) (thickness 0.05)))
+    )
+    (fp_line (start -1.04902 -0.89916) (end 1.04902 -0.89916) (layer F.Fab) (width 0.001))
+    (fp_line (start 1.04902 -0.89916) (end 1.04902 0.89916) (layer F.Fab) (width 0.001))
+    (fp_line (start -1.04902 0.89916) (end 1.04902 0.89916) (layer F.Fab) (width 0.001))
+    (fp_line (start -1.04902 -0.89916) (end -1.04902 0.89916) (layer F.Fab) (width 0.001))
+    (pad 1 smd rect (at -0.7493 0.575 270) (size 0.29972 0.65) (layers F.Cu F.Paste F.Mask)
+      (net 52 "Net-(RP2-Pad1)"))
+    (pad 2 smd rect (at -0.24892 0.575 270) (size 0.29972 0.65) (layers F.Cu F.Paste F.Mask)
+      (net 30 PMS_RX))
+    (pad 3 smd rect (at 0.24892 0.575 270) (size 0.29972 0.65) (layers F.Cu F.Paste F.Mask)
+      (net 29 PMS_TX))
+    (pad 4 smd rect (at 0.7493 0.575 270) (size 0.29972 0.65) (layers F.Cu F.Paste F.Mask)
+      (net 53 "Net-(RP2-Pad4)"))
+    (pad 5 smd rect (at 0.7493 -0.575 90) (size 0.29972 0.65) (layers F.Cu F.Paste F.Mask)
+      (net 54 "Net-(RP2-Pad5)"))
+    (pad 6 smd rect (at 0.24892 -0.575 90) (size 0.29972 0.65) (layers F.Cu F.Paste F.Mask)
+      (net 57 "Net-(RP2-Pad6)"))
+    (pad 7 smd rect (at -0.24892 -0.575 90) (size 0.29972 0.65) (layers F.Cu F.Paste F.Mask)
+      (net 58 "Net-(RP2-Pad7)"))
+    (pad 8 smd rect (at -0.7493 -0.575 90) (size 0.29972 0.65) (layers F.Cu F.Paste F.Mask)
+      (net 55 "Net-(RP2-Pad8)"))
+    (model Resistors_SMD/R_4x0402.wrl
+      (at (xyz 0 0 0))
+      (scale (xyz 1 1 1))
+      (rotate (xyz 0 0 90))
+    )
+  )
